File: ESP32-S3 Stick.kicad_pcb (KiCad board)
At the start: 4 copper layers, 23.1 x 84.2 mm, 43 parts, among them J1 USB_C_Receptacle_USB2.0_16P, J2 Header 22pin, J3 Header 22pin, Q1 DMP2045U-7, SW1 Tactile SW, SW2 Tactile SW, U1 ESP32-S3-WROOM-1, U2 USBLC6-2SC6, U3 MCP73831-2-OT, U4 TPS629210, U5 RV-3028-C7

Commit message: Fixed Broken Symbols
Parts:
- R14: renamed from R11; value 619K -> 619K/0.1%
- R15: renamed from R12; value 137K -> 137K/0.1%
- renumbered C2 to C1, C4 to C2, C6 to C3, C7 to C4, C8 to C6, C9 to C7, C10 to C8, C11 to C9, D3 to D2, D2 to D3, R5 to R1, R7 to R10, R13 to R11, R8 to R12, R10 to R13, R6 to R4, R4 to R5, R9 to R6, R14 to R7, R15 to R8, R16 to R9, U5 to U4, U4 to U5
Connections:
- D2 pad 2: Net-(D3-A) -> Net-(D2-A)
- D3 pad 2: Net-(D2-A) -> Net-(D3-A)

Commit message: Fixed and remapped symbols
Parts:
- R10: value 5.1K -> 10K
- R12, R6: value 10K -> 5.1K
Connections:
- R12 pad 2: Net-(D2-A) -> Net-(D3-A)
- R6 pad 2: Net-(D3-A) -> Net-(D2-A)

Commit message: Fix Silkscreen and re-create fab. files
Other:
- board text added: "SDA-14 SCL-13"
- board text removed: "SDA-13 SCL-14"
Changed lines of the file:
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@@
 			(pdf_back_fp_property_popups yes)
 			(pdf_metadata yes)
-			(pdf_single_document no)
+			(pdf_single_document yes)
 			(dxfpolygonmode yes)
 			(dxfimperialunits yes)
@@
 			(crossoutdnponfab yes)
 			(subtractmaskfromsilk no)
-			(outputformat 5)
+			(outputformat 4)
 			(mirror no)
 			(drillshape 0)
@@
 		(layer "Edge.Cuts")
 	)
-	(gr_text "SDA-13\nSCL-14"
+	(gr_text "SDA-14\nSCL-13"
 		(at 53.6 69.5 0)
 		(layer "F.SilkS")
@@
 	)
 	(segment
+		(start 52.5125 102.67)
+		(end 52.7 102.4825)
+		(width 0.5)
+		(layer "F.Cu")
+		(net "Net-(U3-PROG)")
+	)
+	(segment
+		(start 51.2 102.67)
+		(end 52.5125 102.67)
+		(width 0.5)
+		(layer "F.Cu")
+		(net "Net-(U3-PROG)")
+	)
+	(segment
 		(start 56.475 110.5)
 		(end 56.475 111.9625)
@@
 	)
 	(segment
-		(start 52.5125 102.67)
-		(end 52.7 102.4825)
-		(width 0.5)
-		(layer "F.Cu")
-		(net "Net-(U3-PROG)")
-	)
-	(segment
-		(start 51.2 102.67)
-		(end 52.5125 102.67)
-		(width 0.5)
-		(layer "F.Cu")
-		(net "Net-(U3-PROG)")
-	)
-	(segment
